File: kicad/Eurorack-AS3330-Dual-Lin-Exp-VCA.kicad_sch (KiCad schematic)
At the start: 30 parts, among them U1 AS3330, U2 TL072

Commit message: Added Schematic revision 0.1.1
Parts:
- added C11: 100pF, symbol Device:C
- R1: value 680R -> 560R
- R11, R7: value 150K -> 120K
Connections:
- net Signal Output 1: now also C11.2
- net at R8.1, U1.1 (Iout1), U2.2 (-): now also C11.1
Other:
- note added: "* NOTES * 1) RB should be 120K for a 100uA reference current 2) CV inputs must be normalled to VCC (Digisound) 3) Exp input should be inverted (Digisound) 4) Lin input is a summing node 5) a -10V input would fully attenuate the signal 6) 1nF or larger 7) @15V, 680R, 22mA 7) @12V, 560R, 21.4mA 8) IDLE, @6.8K, class AB, 7uA (Digisound)"
- note added: "*2,3"
- note added: "*2,4,5"
- note added: "*6"
- note added: "*7"
- note added: "*8"
- note added: "1*"
- note added: "10V at the linear control input through the 100K resistor will be at unity gain. 0V would be at -80dB? -10V would be at max attenuation which is -110dB"
Changed lines of the file:
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@@
   (title_block
     (title "Eurorack AS3330 Dual Linear/Exponential VCA")
-    (date "2024-01-27")
-    (rev "0.1.0")
+    (date "2024-01-28")
+    (rev "0.1.1")
     (company "DIYSynthMNL")
     (comment 1 "This version is a prototype")
@@
   (junction (at 148.59 149.86) (diameter 0) (color 0 0 0 0)
   )
+  (junction (at 107.95 59.69) (diameter 0) (color 0 0 0 0)
+  )
   (junction (at 107.95 67.31) (diameter 0) (color 0 0 0 0)
+  )
+  (junction (at 92.71 59.69) (diameter 0) (color 0 0 0 0)
   )
   (junction (at 67.31 187.96) (diameter 0) (color 0 0 0 0)
@@
     (stroke (width 0) (type default))
   )
+  (wire (pts (xy 107.95 53.34) (xy 107.95 59.69))
+    (stroke (width 0) (type default))
+  )
   (wire (pts (xy 41.91 172.72) (xy 41.91 162.56))
     (stroke (width 0) (type default))
@@
   )
   (wire (pts (xy 199.39 83.82) (xy 199.39 76.2))
+    (stroke (width 0) (type default))
+  )
+  (wire (pts (xy 104.14 53.34) (xy 107.95 53.34))
     (stroke (width 0) (type default))
   )
@@
     (stroke (width 0) (type default))
   )
+  (wire (pts (xy 96.52 53.34) (xy 92.71 53.34))
+    (stroke (width 0) (type default))
+  )
   (wire (pts (xy 151.13 172.72) (xy 156.21 172.72))
     (stroke (width 0) (type default))
@@
     (stroke (width 0) (type default))
   )
+  (wire (pts (xy 92.71 53.34) (xy 92.71 59.69))
+    (stroke (width 0) (type default))
+  )
   (wire (pts (xy 113.03 158.75) (xy 115.57 158.75))
     (stroke (width 0) (type default))
@@
     (effects (font (size 1.27 1.27)) (justify left bottom))
   )
+  (text "*2,4,5" (at 19.05 33.02 0)
+    (effects (font (size 1.27 1.27)) (justify left bottom))
+  )
+  (text "*8" (at 149.86 152.4 0)
+    (effects (font (size 1.27 1.27)) (justify left bottom))
+  )
   (text "Iin" (at 57.15 64.77 0)
     (effects (font (size 1.27 1.27)) (justify left bottom))
   )
+  (text "*2,3" (at 20.32 44.45 0)
+    (effects (font (size 1.27 1.27)) (justify left bottom))
+  )
+  (text "*2,3" (at 154.94 44.45 0)
+    (effects (font (size 1.27 1.27)) (justify left bottom))
+  )
+  (text "*6" (at 213.36 50.8 0)
+    (effects (font (size 1.27 1.27)) (justify left bottom))
+  )
+  (text "*7" (at 106.68 167.64 0)
+    (effects (font (size 1.27 1.27)) (justify left bottom))
+  )
   (text "10Vpp" (at 168.91 62.23 0)
     (effects (font (size 1.27 1.27)) (justify left bottom))
   )
+  (text "*2,4,5" (at 153.67 33.02 0)
+    (effects (font (size 1.27 1.27)) (justify left bottom))
+  )
   (text "Iout" (at 222.25 64.77 0)
     (effects (font (size 1.27 1.27)) (justify left bottom))
   )
+  (text "*6" (at 78.74 50.8 0)
+    (effects (font (size 1.27 1.27)) (justify left bottom))
+  )
+  (text "1*" (at 198.12 43.18 0)
+    (effects (font (size 1.27 1.27)) (justify left bottom))
+  )
   (text "Iout" (at 87.63 64.77 0)
+    (effects (font (size 1.27 1.27)) (justify left bottom))
+  )
+  (text "1*" (at 63.5 43.18 0)
     (effects (font (size 1.27 1.27)) (justify left bottom))
   )
@@
     (effects (font (size 1.27 1.27)) (justify left bottom))
   )
+  (text "* NOTES *\n1) RB should be 120K for a 100uA reference current\n2) CV inputs must be normalled to VCC (Digisound)\n3) Exp input should be inverted (Digisound)\n4) Lin input is a summing node\n5) a -10V input would fully attenuate the signal\n6) 1nF or larger\n7) @15V, 680R, 22mA\n7) @12V, 560R, 21.4mA\n8) IDLE, @6.8K, class AB, 7uA (Digisound)"
+    (at 177.8 163.83 0)
+    (effects (font (size 1.27 1.27)) (justify left bottom))
+  )
   (text "REE" (at 106.68 165.1 0)
     (effects (font (size 1.27 1.27)) (justify left bottom))
@@
     (effects (font (size 1.27 1.27)) (justify left bottom))
   )
+  (text "1*" (at 198.12 43.18 0)
+    (effects (font (size 1.27 1.27)) (justify left bottom))
+  )
   (text "Vce" (at 190.5 41.91 0)
     (effects (font (size 1.27 1.27)) (justify left bottom))
@@
   )
   (text "0V to 10V" (at 153.67 27.94 0)
+    (effects (font (size 1.27 1.27)) (justify left bottom))
+  )
+  (text "10V at the linear control input through the 100K resistor will be at unity gain.\n0V would be at -80dB?\n-10V would be at max attenuation which is -110dB"
+    (at 27.94 114.3 0)
     (effects (font (size 1.27 1.27)) (justify left bottom))
   )
@@
       (effects (font (size 1.27 1.27)) (justify left))
     )
-    (property "Value" "680R" (at 115.57 166.37 0)
+    (property "Value" "560R" (at 115.57 166.37 0)
       (effects (font (size 1.27 1.27)) (justify left))
     )
@@
       (effects (font (size 1.27 1.27)) (justify left))
     )
-    (property "Value" "150K" (at 203.2 40.64 0)
+    (property "Value" "120K" (at 203.2 40.64 0)
       (effects (font (size 1.27 1.27)) (justify left))
     )
@@
         (path "/7e0f364c-4839-48e2-a5ac-184d21827e3d"
           (reference "C2") (unit 1)
+        )
+      )
+    )
+  )
+  (symbol (lib_id "Device:C") (at 100.33 53.34 90) (unit 1)
+    (in_bom yes) (on_board yes) (dnp no)
+    (property "Reference" "C11" (at 100.33 46.99 90)
+      (effects (font (size 1.27 1.27)))
+    )
+    (property "Value" "100pF" (at 100.33 49.53 90)
+      (effects (font (size 1.27 1.27)))
+    )
+    (property "Footprint" "" (at 104.14 52.3748 0)
+      (effects (font (size 1.27 1.27)) hide)
+    )
+    (property "Datasheet" "~" (at 100.33 53.34 0)
+      (effects (font (size 1.27 1.27)) hide)
+    )
+    (pin "2")
+    (pin "1")
+    (instances
+      (project "Eurorack-AS3330-Dual-Lin-Exp-VCA"
+        (path "/7e0f364c-4839-48e2-a5ac-184d21827e3d"
+          (reference "C11") (unit 1)
         )
       )
@@
       (effects (font (size 1.27 1.27)) (justify left))
     )
-    (property "Value" "150K" (at 68.58 40.64 0)
+    (property "Value" "120K" (at 68.58 40.64 0)
       (effects (font (size 1.27 1.27)) (justify left))
     )

Commit message: updated schematic rev 0.1.1
Parts:
- added C5: 100pF, symbol Device:C
- renumbered C6 to C1, C10 to C11, C11 to C2, C7 to C3, C8 to C4, C9 to C6, C5 to C7, C1 to C8, C2 to C9, R6 to R1, R12 to R10, R13 to R11, R14 to R12, R2 to R13, R1 to R14, R5 to R2, R7 to R3, R8 to R5, R3 to R6, R9 to R7, R10 to R8, R11 to R9
Connections:
- net Signal Output 2: now also C5.2
- net at R11.1, U1.16 (Iout2), U2.6 (-): now also C5.1

Commit message: added schematic revision 0.1.3
Parts:
- added C13, C14: 100nF, symbol Device:C
- added D3, D4, D5, D6, D7, D8: BAT42, symbol Device:D_Schottky
- added J3: CV1 In, DIYSynthMNL:AudioJack_3.5mm_long_pads, symbol DIYSynthMNL:PJ3001F
- added J4: CV2 In, DIYSynthMNL:AudioJack_3.5mm_long_pads, symbol DIYSynthMNL:PJ3001F
- added J5: Sig In 2, DIYSynthMNL:AudioJack_3.5mm_long_pads, symbol DIYSynthMNL:PJ3001F
- added J6: Sig In 1, DIYSynthMNL:AudioJack_3.5mm_long_pads, symbol DIYSynthMNL:PJ3001F
- added J7, J8: Sig out 1, DIYSynthMNL:AudioJack_3.5mm_long_pads, symbol DIYSynthMNL:PJ3001F
- added R15, R16, R17, R18, R19, R20, R21, R22, R24, R25, R29, R30, R31, R32, R33, R34, R35, R36, R39, R40: 100K, symbol Device:R
- added R23, R28: 200K, symbol Device:R
- added R26, R27, R37, R38: 4.7K, symbol Device:R
- added RV1, RV3, RV4, RV6: 100K, symbol Device:R_Potentiometer
- added RV2, RV5: 10K, symbol Device:R_Potentiometer
- added U3, U4: TL074, symbol Amplifier_Operational:TL074
- R11, R5: value 51K -> 100K
- R13: value 6.8K -> 68K
Connections:
- net +12V: now also C13.1, C14.1, U3.4 (V+), U4.4 (V+)
- net -12V: now also C13.2, C14.2, U3.11 (V-), U4.11 (V-)
- net Exponential CV Input 1: now also R26.2, RV3.3
- net Exponential CV Input 2: now also R37.2, RV6.3
- net GND: now also D5.2 (A), D8.2 (A), J3.S, J4.S, J5.S, J6.S, J7.S, J8.S, R24.2, R40.2, RV1.1, RV2.3, RV3.2, RV4.1, RV5.3, RV6.2, U3.10 (+), U3.3 (+), U3.5 (+), U4.10 (+), U4.3 (+), U4.5 (+)
- net Linear CV Input 1: now also D5.1 (K), R27.2, RV3.1
- net Linear CV Input 2: now also D8.1 (K), R38.2, RV6.1
- net Signal Input 1: now also J5.TN, J6.T
- net Signal Input 2: now also J5.T
- net Signal Output 1: now also J7.T
- net Signal Output 2: now also J8.T
- new net: R30.2, R34.1, U3.12 (+), U3.7
- new net: D7.2 (A), R28.1, R34.2, R36.2, U3.9 (-)
- new net: R18.2, R19.2, R20.1, U4.6 (-)
- new net: R20.2, R21.1, U4.12 (+), U4.7
- new net: R30.1, R32.2, R35.2, U3.6 (-)
- new net: R15.1, RV1.2
- new net: D4.2 (A), R21.2, R22.2, R23.1, U4.9 (-)
- new net: D6.2 (A), D7.1 (K), U3.8
- new net: R24.1, R25.1, U4.13 (-)
- new net: R25.2, R27.1, U4.14
- new net: R15.2, R16.2, R17.1, U4.2 (-)
- new net: R39.1, R40.1, U3.13 (-)
- new net: R29.2, R32.1, U3.1
- new net: R29.1, R31.2, R33.2, U3.2 (-)
- new net: D3.2 (A), D4.1 (K), U4.8
- new net: R16.1, RV2.2
- new net: R33.1, RV5.2
- new net: D6.1 (K), R28.2, R37.1
- new net: R17.2, R18.1, U4.1
- new net: R31.1, RV4.2
- new net: D3.1 (K), R23.2, R26.1
- new net: R38.1, R39.2, U3.14
- new net -5V: R19.1, R22.1, R35.1, R36.1, RV2.1, RV5.1
- new net CV1 IN: J3.T, J4.TN, RV1.3
- new net CV2 IN: J4.T, RV4.3
- no-connect marks 6 -> 10
Other:
- note added: ""Pan" between linear and exponential"
- note added: "* NOTES * 1) RB should be 120K for a 100uA reference current 2) CV inputs must be normalled to VCC (Digisound) 3) Exp input should be inverted (Digisound) 4) Lin input is a summing node 5) a -10V input would fully attenuate the signal 6) 1nF or larger 7) @15V, 680R, 22mA 7) @12V, 560R, 21.4mA 8) IDLE, @68K, Class A"
- note added: "CV Attenuation knob"
- note added: "CV Offset knob"
- note added: "CV Scaling and Lin/Exp control 1"
- note added: "CV Scaling and Lin/Exp control 2"
- note added: "Control inputs (single input/either or): Linear (Exp input must be at 0V or unity gain): - 10V at the linear CV input through the 100K resistor will be at unity gain. - 0V would be max attenuation. Exponential (Linear input must be at 10V or unity gain): - 0V at the exponential CV input through the 33K resistor will be at unity gain. - 10V would be max attenuation."
- note added: "Flexible input levels with the use of two knobs: 10Vpp 0V to 5V 0V to 10V"
- note added: "Lin/Exp knob"
- note added: "Offset + Invert back to original phase"
- note added: "Offset+invert"
- note added: "Offset, Double the voltage to 0 to 10V, cut negative voltages, invert for exponential cv in"
- note removed: "* NOTES * 1) RB should be 120K for a 100uA reference current 2) CV inputs must be normalled to VCC (Digisound) 3) Exp input should be inverted (Digisound) 4) Lin input is a summing node 5) a -10V input would fully attenuate the signal 6) 1nF or larger 7) @15V, 680R, 22mA 7) @12V, 560R, 21.4mA 8) IDLE, @6.8K, class AB, 7uA (Digisound)"
- note removed: "10V at the linear control input through the 100K resistor will be at unity gain. 0V would be at -80dB? -10V would be at max attenuation which is -110dB"
- moved on the sheet: C1, C11, C2, C3, C4, C5, C6, C7, C8, C9, C?, D?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

Commit message: Added Schematic revision 0.1.4
Parts:
- removed J4: CV2 In, DIYSynthMNL:AudioJack_3.5mm_long_pads, symbol DIYSynthMNL:PJ3001F
- removed R18, R19, R20, R35, R36: 100K, symbol Device:R
- removed unit 5 of U4
- removed unit 2 of U4
- added C10, C11, C12, C21, C7, C8, C9: 100pF, symbol Device:C
- added D3, D4: BAT42, symbol Device:D_Schottky
- added J6: CV2 In, DIYSynthMNL:AudioJack_3.5mm_long_pads, symbol DIYSynthMNL:PJ3001F
- added J9: Mix Out, DIYSynthMNL:AudioJack_3.5mm_long_pads, symbol DIYSynthMNL:PJ3001F
- added R14, R7: 1K, symbol Device:R
- added R25: 200K, symbol Device:R
- added R26: 180K, symbol Device:R
- added R27: 100K, symbol Device:R
- added RV7: 10K, symbol Device:R_Potentiometer_Trim
- added TP1: -5VREF, symbol Connector:TestPoint
- added unit 2 of U3
- added unit 5 of U3
- R16: renamed from R17; value 100K -> 180K
- R18: renamed from R26; value 4.7K -> 6.8K
- R22: renamed from R27; value 4.7K -> 6.8K
- R28: value 200K -> 6.8K
- R32: value 100K -> 6.8K
- R37, R38: value 4.7K -> 100K
- R40: value 100K -> 1K
- RV2: renamed from RV3; value 100K -> 10K
- RV6: value 100K -> 10K
- renumbered C7 to C15, C8 to C16, C9 to C17, C11 to C18, C14 to C19, C13 to C20, D3 to D1, D4 to D2, J6 to J1, J7 to J2, J5 to J3, J8 to J4, J3 to J5, R9 to R10, R10 to R11, R11 to R12, R12 to R13, R23 to R15, R15 to R17, R16 to R19, R21 to R20, R22 to R21, R25 to R23, R13 to R35, R14 to R36, R7 to R8, R8 to R9, RV2 to RV3, U3 to U2, U4 to U2, U2 to U4
Connections:
- net +12V: now also U3.4 (V+)
- net -12V: now also RV7.3, U3.11 (V-)
- net CV1 IN: now also J6.TN
- net CV2 IN: now also J6.T
- net Exponential CV Input 1: now also R23.2, C9.2, D4.1 (K); no longer R18.2, RV2.3
- net Exponential CV Input 2: now also D8.1 (K), R33.2, C12.2; no longer R37.2, RV6.3
- net GND: now also R34.2, RV5.2, RV6.3, U2.12 (+), U3.12 (+), J6.S, J9.S, RV7.1, U3.5 (+); no longer D5.2 (A), D8.2 (A), R40.2, RV5.3, RV6.2, U2.10 (+), U3.10 (+), U4.3 (+)
- net Linear CV Input 1: now also D1.1 (K), R15.2, C7.2; no longer D5.1 (K), R22.2, RV2.1
- net Linear CV Input 2: now also D5.1 (K), C10.2, R25.2; no longer D8.1 (K), R38.2, RV6.1
- net Signal Output 1: now also R37.1, U2.14, R7.1; no longer J2.T, U4.1
- net Signal Output 2: now also R39.1, U3.14, R14.1; no longer J4.T, U4.7
- net at C2.1, R5.1, U1.1 (Iout1): now also U2.13 (-); no longer U4.2 (-)
- net at D7.2 (A), U3.9 (-): now also R33.1, R34.1, C12.1; no longer R28.1, R34.2
- net at R20.1: now also R18.2, RV2.3; no longer U2.12 (+)
- net at D2.2 (A), R15.1, R20.2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: now also U2.6 (-), C7.1; no longer U2.9 (-)
- net at D7.1 (K), U3.8: now also D8.2 (A); no longer D6.2 (A)
- net at R23.1, R24.1: now also U2.9 (-), C9.1, D3.2 (A); no longer U2.13 (-)
- net at C5.1, R12.1, U1.16 (Iout2): now also U3.13 (-); no longer U4.6 (-)
- net at R16.1, R17.2, R19.2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: now also C8.1
- net at R32.1, U3.1: now also R28.1, C11.2, R26.2; no longer R29.2
- net at D1.2 (A), D2.1 (K): now also U2.7; no longer U2.8
- net at R16.2, U2.1: now also R18.1, R22.1, C8.2
- net at RV4.2: now also R27.1; no longer R31.1
- net at R38.1, R39.2: now also R37.2, U4.6 (-), C21.1; no longer U3.14
- net -5V renamed -5VRef
- net -5VRef: now also R31.1, RV6.1, U4.1, U4.2 (-), TP1.1; no longer RV5.1
- new net: R29.1, RV6.2
- new net: C11.1, R26.1, R27.2, R29.2, U3.2 (-)
- new net: C10.1, D6.2 (A), R25.1, R30.2, R31.2, U3.6 (-)
- new net: D5.2 (A), D6.1 (K), U3.7
- new net: C21.2, R38.2, R40.1, U4.7
- new net: RV7.2, U4.3 (+)
- new net: J9.T, R40.2
- new net: R22.2, RV2.1, U2.10 (+)
- new net: R32.2, RV5.1, U3.10 (+)
- new net: R28.2, R30.1, RV5.3
- new net: D3.1 (K), D4.2 (A), U2.8
- new net: J4.T, R14.2
- new net: J2.T, R7.2
- no-connect marks 10 -> 11
Other:
- note added: "-5V reference"
- note added: "3330 power and idle"
- note added: "Is inverted from signal outputs"
- note added: "Mix out"
- note added: "Offset+invert+gain"
- note added: "Offset, Double the voltage to 0 to 10V, cut negative voltages, invert for linear cv"
- note added: "Op amp power and decoupling"
- note removed: "Offset + Invert back to original phase"
- note removed: "Offset+invert"
- note removed: "Offset, Double the voltage to 0 to 10V, cut negative voltages, invert for exponential cv in"
- moved on the sheet: J2, J4, R18, R22, R23, R24, RV2, U2B, U2C, U2D, U4A, U4B

Commit message: added schematic rev0.1.5
Parts:
- added C22: 100nF, symbol Device:C
- added D11: HI1, symbol Device:LED
- added D12: LO1, symbol Device:LED
- added D13: HI2, symbol Device:LED
- added D14: LO2, symbol Device:LED
- added R41, R42, R45, R46: 1M, symbol Device:R
- added R43, R44: ~, symbol Device:R
- added U5: TL072, symbol Amplifier_Operational:TL072
Connections:
- net +12V: now also C22.1, U5.8 (V+)
- net -12V: now also C22.2, U5.4 (V-)
- net GND: now also R42.1, R43.1, R44.1, R46.1, U5.3 (+), U5.5 (+); no longer U2.12 (+), U3.12 (+)
- net Signal Output 1: now also U5.1; no longer U2.14
- net Signal Output 2: now also U5.7; no longer U3.14
- net at C2.1, R5.1, U1.1 (Iout1): now also U5.2 (-); no longer U2.13 (-)
- net LED1: now reaches R17.1, RV1.2
- net LED1: now also R41.1
- net LED2: now reaches R27.1, RV4.2
- net LED2: now also R45.1
- net at C5.1, R12.1, U1.16 (Iout2): now also U5.6 (-); no longer U3.13 (-)
- new net: D13.2 (A), D14.1 (K), U3.14
- new net: D13.1 (K), D14.2 (A), R44.2, U3.13 (-)
- new net: R45.2, R46.2, U3.12 (+)
- new net: D11.2 (A), D12.1 (K), U2.14
- new net: D11.1 (K), D12.2 (A), R43.2, U2.13 (-)
- new net: R41.2, R42.2, U2.12 (+)
Other:
- note added: "Knob 0% (Left) = Linear Knob 100% (Right) = Exponential"
- note added: "LED Indicator"
- moved on the sheet: C18, C19, C20, RV7, TP1, U2D, U2E, U3D, U3E, U4A, U4C

Commit message: Schematic rev 0.1.5 updated
Parts:
- added C23: 100nF, symbol Device:C
- added R41, R45: 100K, symbol Device:R
- added unit 1 of U5
- added unit 2 of U5
- added unit 3 of U6
- renumbered C21 to C13, C15 to C16, C16 to C17, C17 to C18, C22 to C19, C18 to C20, C19 to C21, C20 to C22, D7 to D10, D14 to D11, D8 to D12, D11 to D3, D3 to D4, D12 to D5, D4 to D6, D5 to D7, D6 to D8, D13 to D9, J9 to J7, R43 to R23, R23 to R24, R41 to R25, R42 to R26, R24 to R27, R25 to R28, R26 to R29, R27 to R30, R28 to R31, R29 to R32, R30 to R33, R31 to R34, R32 to R35, R44 to R36, R33 to R37, R45 to R38, R46 to R39, R34 to R40, R37 to R42, R38 to R43, R39 to R44, R40 to R46, R35 to R47, R36 to R48, U5 to U2, U2 to U3, U3 to U4, U4 to U5, U4 to U6
Connections:
- net +12V: now also C23.1, U6.8 (V+)
- net -12V: now also C23.2, U6.4 (V-)
- net GND: now also U5.3 (+), U5.5 (+)
- net at C13.1, R42.2, R43.1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: now also U5.2 (-); no longer U6.6 (-)
- net at C13.2, R43.2: now also R45.1, U5.1; no longer R46.1, U6.7
- new net: U6.6 (-), U6.7
- new net: R41.2, R46.1, U5.7
- new net: R41.1, R45.2, U5.6 (-)
Other:
- note removed: "Is inverted from signal outputs"
- moved on the sheet: C19, C20, C21, C22, J7, R46, RV7, TP1, U2C, U3E, U4E, U5C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
