File: kicad/Eurorack-AS3330-Dual-Lin-Exp-VCA.kicad_sch (KiCad schematic)
At the start: 108 parts, among them J1 Sig In 1, J2 Sig out 1, J3 Sig In 2, J4 Sig out 1, J5 CV1 In, J6 CV2 In, J7 Mix Out, U1 AS3330, U2 TL072, U3 TL074, U4 TL074, U5 TL072, U6 TL072

Commit message: Added schematic rev 0.1.6
Parts:
- removed D11: LO2, symbol Device:LED
- removed D3: HI1, symbol Device:LED
- removed D5: LO1, symbol Device:LED
- removed D9: HI2, symbol Device:LED
- added D15, D3: LED_Dual_Bidirectional, symbol Device:LED_Dual_Bidirectional
Connections:
- net at U4.14: now also D3.1 (KA)
- net at R36.2, U4.13 (-): now also D3.2 (AK)
- net at U3.14: now also D15.1 (KA)
- net at R23.2, U3.13 (-): now also D15.2 (AK)
Changed lines of the file:
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@@
   (title_block
     (title "Eurorack AS3330 Dual Linear/Exponential VCA")
-    (date "2024-02-02")
-    (rev "0.1.5")
+    (date "2024-02-13")
+    (rev "0.1.6")
     (company "DIYSynthMNL")
     (comment 1 "This version is a prototype")
@@
   (junction (at 173.99 182.245) (diameter 0) (color 0 0 0 0)
   )
-  (junction (at 102.87 92.71) (diameter 0) (color 0 0 0 0)
-  )
   (junction (at 106.68 151.765) (diameter 0) (color 0 0 0 0)
   )
@@
   (junction (at 173.99 262.255) (diameter 0) (color 0 0 0 0)
   )
-  (junction (at 176.53 142.875) (diameter 0) (color 0 0 0 0)
+  (junction (at 102.87 92.71) (diameter 0) (color 0 0 0 0)
   )
-  (junction (at 122.555 184.785) (diameter 0) (color 0 0 0 0)
+  (junction (at 176.53 142.875) (diameter 0) (color 0 0 0 0)
   )
   (junction (at 176.53 64.77) (diameter 0) (color 0 0 0 0)
@@
   (junction (at 135.89 254) (diameter 0) (color 0 0 0 0)
   )
-  (junction (at 118.11 92.71) (diameter 0) (color 0 0 0 0)
-  )
   (junction (at 106.045 195.58) (diameter 0) (color 0 0 0 0)
   )
@@
     (stroke (width 0) (type default))
   )
-  (wire (pts (xy 122.555 184.785) (xy 122.555 180.34))
+  (wire (pts (xy 122.555 184.785) (xy 122.555 193.04))
     (stroke (width 0) (type default))
   )
@@
     (stroke (width 0) (type default))
   )
-  (wire (pts (xy 107.315 180.34) (xy 111.125 180.34))
-    (stroke (width 0) (type default))
-  )
   (wire (pts (xy 314.325 20.32) (xy 318.135 20.32))
     (stroke (width 0) (type default))
@@
     (stroke (width 0) (type default))
   )
-  (wire (pts (xy 118.11 88.265) (xy 114.3 88.265))
-    (stroke (width 0) (type default))
-  )
   (wire (pts (xy 41.91 259.08) (xy 41.91 248.92))
     (stroke (width 0) (type default))
@@
     (stroke (width 0) (type default))
   )
-  (wire (pts (xy 122.555 180.34) (xy 118.745 180.34))
-    (stroke (width 0) (type default))
-  )
   (wire (pts (xy 67.31 264.16) (xy 67.31 266.7))
     (stroke (width 0) (type default))
@@
     (stroke (width 0) (type default))
   )
-  (wire (pts (xy 111.125 184.785) (xy 107.315 184.785))
-    (stroke (width 0) (type default))
-  )
   (wire (pts (xy 255.27 66.04) (xy 278.13 66.04))
     (stroke (width 0) (type default))
@@
     (stroke (width 0) (type default))
   )
-  (wire (pts (xy 102.87 92.71) (xy 102.87 88.265))
-    (stroke (width 0) (type default))
-  )
   (wire (pts (xy 187.96 136.525) (xy 200.66 136.525))
     (stroke (width 0) (type default))
@@
     (stroke (width 0) (type default))
   )
-  (wire (pts (xy 118.11 92.71) (xy 118.11 88.265))
-    (stroke (width 0) (type default))
-  )
   (wire (pts (xy 327.66 83.82) (xy 327.66 88.9))
     (stroke (width 0) (type default))
@@
     (stroke (width 0) (type default))
   )
-  (wire (pts (xy 102.87 88.265) (xy 106.68 88.265))
-    (stroke (width 0) (type default))
-  )
   (wire (pts (xy 69.85 147.955) (xy 83.82 147.955))
     (stroke (width 0) (type default))
@@
     (stroke (width 0) (type default))
   )
-  (wire (pts (xy 122.555 193.04) (xy 122.555 184.785))
-    (stroke (width 0) (type default))
-  )
   (wire (pts (xy 173.99 182.245) (xy 179.705 182.245))
     (stroke (width 0) (type default))
@@
     (stroke (width 0) (type default))
   )
-  (wire (pts (xy 114.3 92.71) (xy 118.11 92.71))
-    (stroke (width 0) (type default))
-  )
   (wire (pts (xy 293.37 151.13) (xy 293.37 162.56))
     (stroke (width 0) (type default))
@@
     (stroke (width 0) (type default))
   )
-  (wire (pts (xy 118.745 184.785) (xy 122.555 184.785))
-    (stroke (width 0) (type default))
-  )
   (wire (pts (xy 187.96 142.875) (xy 191.77 142.875))
     (stroke (width 0) (type default))
@@
     (stroke (width 0) (type default))
   )
-  (wire (pts (xy 106.68 92.71) (xy 102.87 92.71))
-    (stroke (width 0) (type default))
-  )
   (wire (pts (xy 194.945 247.015) (xy 188.595 247.015))
     (stroke (width 0) (type default))
   )
-  (wire (pts (xy 107.315 184.785) (xy 107.315 180.34))
-    (stroke (width 0) (type default))
-  )
   (wire (pts (xy 304.8 73.66) (xy 304.8 76.2))
     (stroke (width 0) (type default))
@@
     )
   )
-  (symbol (lib_id "Device:LED") (at 114.935 184.785 180) (unit 1)
-    (in_bom yes) (on_board yes) (dnp no)
-    (property "Reference" "D11" (at 127 184.15 0)
-      (effects (font (size 1.27 1.27)))
-    )
-    (property "Value" "LO2" (at 127 186.69 0)
-      (effects (font (size 1.27 1.27)))
-    )
-    (property "Footprint" "" (at 114.935 184.785 0)
-      (effects (font (size 1.27 1.27)) hide)
-    )
-    (property "Datasheet" "~" (at 114.935 184.785 0)
-      (effects (font (size 1.27 1.27)) hide)
-    )
-    (pin "1")
-    (pin "2")
-    (instances
-      (project "Eurorack-AS3330-Dual-Lin-Exp-VCA"
-        (path "/7e0f364c-4839-48e2-a5ac-184d21827e3d"
-          (reference "D11") (unit 1)
-        )
-      )
-    )
-  )
   (symbol (lib_id "power:PWR_FLAG") (at 83.82 259.08 0) (unit 1)
     (in_bom yes) (on_board yes) (dnp no) (fields_autoplaced)
@@
     )
   )
-  (symbol (lib_id "Device:LED") (at 110.49 92.71 180) (unit 1)
-    (in_bom yes) (on_board yes) (dnp no)
-    (property "Reference" "D5" (at 122.555 92.075 0)
-      (effects (font (size 1.27 1.27)))
-    )
-    (property "Value" "LO1" (at 122.555 94.615 0)
-      (effects (font (size 1.27 1.27)))
-    )
-    (property "Footprint" "" (at 110.49 92.71 0)
-      (effects (font (size 1.27 1.27)) hide)
-    )
-    (property "Datasheet" "~" (at 110.49 92.71 0)
-      (effects (font (size 1.27 1.27)) hide)
-    )
-    (pin "1")
-    (pin "2")
-    (instances
-      (project "Eurorack-AS3330-Dual-Lin-Exp-VCA"
-        (path "/7e0f364c-4839-48e2-a5ac-184d21827e3d"
-          (reference "D5") (unit 1)
-        )
-      )
-    )
-  )
   (symbol (lib_id "power:GND") (at 110.49 156.845 0) (unit 1)
     (in_bom yes) (on_board yes) (dnp no) (fields_autoplaced)
@@
     )
   )
+  (symbol (lib_id "Device:LED_Dual_Bidirectional") (at 110.49 92.71 0) (unit 1)
+    (in_bom yes) (on_board yes) (dnp no) (fields_autoplaced)
+    (property "Reference" "D15" (at 110.9853 81.915 0)
+      (effects (font (size 1.27 1.27)))
+    )
+    (property "Value" "LED_Dual_Bidirectional" (at 110.9853 84.455 0)
+      (effects (font (size 1.27 1.27)))
+    )
+    (property "Footprint" "" (at 110.49 92.71 0)
+      (effects (font (size 1.27 1.27)) hide)
+    )
+    (property "Datasheet" "~" (at 110.49 92.71 0)
+      (effects (font (size 1.27 1.27)) hide)
+    )
+    (pin "1")
+    (pin "2")
+    (instances
+      (project "Eurorack-AS3330-Dual-Lin-Exp-VCA"
+        (path "/7e0f364c-4839-48e2-a5ac-184d21827e3d"
+          (reference "D15") (unit 1)
+        )
+      )
+    )
+  )
   (symbol (lib_id "Device:R") (at 132.08 168.275 90) (unit 1)
     (in_bom yes) (on_board yes) (dnp no)
@@
     )
   )
-  (symbol (lib_id "Device:LED") (at 110.49 88.265 0) (unit 1)
-    (in_bom yes) (on_board yes) (dnp no)
-    (property "Reference" "D3" (at 122.555 86.36 0)
-      (effects (font (size 1.27 1.27)))
-    )
-    (property "Value" "HI1" (at 122.555 88.9 0)
-      (effects (font (size 1.27 1.27)))
-    )
-    (property "Footprint" "" (at 110.49 88.265 0)
-      (effects (font (size 1.27 1.27)) hide)
-    )
-    (property "Datasheet" "~" (at 110.49 88.265 0)
-      (effects (font (size 1.27 1.27)) hide)
-    )
-    (pin "1")
-    (pin "2")
-    (instances
-      (project "Eurorack-AS3330-Dual-Lin-Exp-VCA"
-        (path "/7e0f364c-4839-48e2-a5ac-184d21827e3d"
-          (reference "D3") (unit 1)
-        )
-      )
-    )
-  )
   (symbol (lib_id "Device:R") (at 365.76 91.44 90) (unit 1)
     (in_bom yes) (on_board yes) (dnp no)
@@
     )
   )
-  (symbol (lib_id "Device:LED") (at 114.935 180.34 0) (unit 1)
-    (in_bom yes) (on_board yes) (dnp no)
-    (property "Reference" "D9" (at 127 178.435 0)
-      (effects (font (size 1.27 1.27)))
-    )
-    (property "Value" "HI2" (at 127 180.975 0)
-      (effects (font (size 1.27 1.27)))
-    )
-    (property "Footprint" "" (at 114.935 180.34 0)
-      (effects (font (size 1.27 1.27)) hide)
-    )
-    (property "Datasheet" "~" (at 114.935 180.34 0)
-      (effects (font (size 1.27 1.27)) hide)
-    )
-    (pin "1")
-    (pin "2")
-    (instances
-      (project "Eurorack-AS3330-Dual-Lin-Exp-VCA"
-        (path "/7e0f364c-4839-48e2-a5ac-184d21827e3d"
-          (reference "D9") (unit 1)
-        )
-      )
-    )
-  )
   (symbol (lib_id "DIYSynthMNL:PJ3001F") (at 260.35 173.99 0) (mirror x) (unit 1)
     (in_bom yes) (on_board yes) (dnp no) (fields_autoplaced)
@@
         )
       )
+    )
+  )
+  (symbol (lib_id "Device:LED_Dual_Bidirectional") (at 114.935 184.785 0) (unit 1)
+    (in_bom yes) (on_board yes) (dnp no) (fields_autoplaced)
+    (property "Reference" "D3" (at 115.4303 173.99 0)
+      (effects (font (size 1.27 1.27)))
+    )
+    (property "Value" "LED_Dual_Bidirectional" (at 115.4303 176.53 0)
+      (effects (font (size 1.27 1.27)))
+    )
+    (property "Footprint" "" (at 114.935 184.785 0)
+      (effects (font (size 1.27 1.27)) hide)
+    )
+    (property "Datasheet" "~" (at 114.935 184.785 0)
+      (effects (font (size 1.27 1.27)) hide)
+    )
+    (pin "1")
+    (pin "2")
+    (instances
+      (project "Eurorack-AS3330-Dual-Lin-Exp-VCA"
+        (path "/7e0f364c-4839-48e2-a5ac-184d21827e3d"
+          (reference "D3") (unit 1)
+        )
+      )

Commit message: added schem rev 0.1.7
Parts:
- removed J4: Sig out 1, DIYSynthMNL:AudioJack_3.5mm_long_pads, symbol DIYSynthMNL:PJ3001F
- removed J7: Mix Out, DIYSynthMNL:AudioJack_3.5mm_long_pads, symbol DIYSynthMNL:PJ3001F
- removed R14: 1K, symbol Device:R
- added J12: Sig out 2, DIYSynthMNL:AudioJack_3.5mm_long_pads, symbol DIYSynthMNL:PJ3001F
- added JP1: Mix/VCA4, symbol Jumper:Jumper_3_Bridged12
Connections:
- net GND: now also J12.S
- net Signal Output 2: now also JP1.3 (B)
- net at R46.2: now also J12.T
- net Mix Out: now reaches R41.2, U5.7
- net Mix Out: now also JP1.1 (A); no longer R46.1
- new net: JP1.2 (C), R46.1
- no-connect marks 11 -> 10
Other:
- note added: "Mix"
- note added: "Out 2 Select"
- note removed: "Mix out"
- moved on the sheet: C13, R41, R42, R43, R44, R45, R46, U5A, U5B
